Commit message: Remove fingers from Gazebo as they are not useful and slow down the simulation (and arent actually correctly simulated anyways)

File: pepper_description/urdf/pepper1.0_generated_urdf/pepperGazebo.xacro (robot description, xacro)
@@ -3,5 +3,5 @@
     <!-- MACROS FOR DISABLE LINKS -->
 	<xacro:property name="PI" value="3.14159265359" />
-    <xacro:macro name="DisabledLinks" params="side side_small">
+    <!-- <xacro:macro name="DisabledLinks" params="side side_small">
         <plugin name="${side}Finger11_link" filename="libroboticsgroup_gazebo_disable_link_plugin.so">
             <link>${side}Finger11_link</link>
@@ -49,8 +49,8 @@
             <link>${side_small}_gripper</link>
         </plugin>
-    </xacro:macro>
+    </xacro:macro>  -->
     <!-- MACROS FOR MIMIC JOINTS -->
     <!-- Fingers -->
-    <xacro:macro name="FingerMimics" params="side num">
+ <!--    <xacro:macro name="FingerMimics" params="side num">
         <plugin name="mimic_${side}Finger${num}1" filename="libroboticsgroup_gazebo_mimic_joint_plugin.so">
             <joint>${side}Hand</joint>
@@ -72,5 +72,4 @@
         </plugin>
     </xacro:macro>
-    <!-- Thumbs -->
     <xacro:macro name="ThumbMimics" params="side">
         <plugin name="${side}Thumb1" filename="libroboticsgroup_gazebo_mimic_joint_plugin.so">
@@ -86,5 +85,5 @@
             <offset>${PI/4}</offset>
         </plugin>
-    </xacro:macro>
+    </xacro:macro> -->
     <!-- GAZEBO ROS CONTROL -->
     <gazebo>
@@ -93,5 +92,5 @@
             <robotSimType>gazebo_ros_control/DefaultRobotHWSim</robotSimType>
         </plugin>
-        <xacro:FingerMimics side="L" num="1"/>
+ <!--        <xacro:FingerMimics side="L" num="1"/>
         <xacro:FingerMimics side="L" num="2"/>
         <xacro:FingerMimics side="L" num="3"/>
@@ -104,5 +103,5 @@
         <xacro:ThumbMimics side="R"/>
         <xacro:DisabledLinks side="L" side_small="l"/>
-        <xacro:DisabledLinks side="R" side_small="r"/>
+        <xacro:DisabledLinks side="R" side_small="r"/>  -->
     </gazebo>
     <!-- END OF GAZEBO ROS CONTROL PLUGIN -->
@@ -211,5 +210,5 @@
         <turnGravityOff>true</turnGravityOff>
     </gazebo>
-    <gazebo reference="LFinger11_link">
+<!--     <gazebo reference="LFinger11_link">
         <mu1>0.5</mu1>
         <mu2>0.5</mu2>
@@ -294,5 +293,5 @@
         <selfCollide>false</selfCollide>
         <turnGravityOff>true</turnGravityOff>
-    </gazebo>
+    </gazebo>  -->
     <gazebo reference="Hip">
         <mu1>0.5</mu1>
@@ -340,5 +339,5 @@
         <turnGravityOff>false</turnGravityOff>
     </gazebo>
-    <gazebo reference="RFinger11_link">
+  <!--   <gazebo reference="RFinger11_link">
         <mu1>0.5</mu1>
         <mu2>0.5</mu2>
@@ -423,5 +422,5 @@
         <selfCollide>false</selfCollide>
         <turnGravityOff>true</turnGravityOff>
-    </gazebo>
+    </gazebo> -->
 <!--
         RGB CAMERAS:

File: pepper_description/urdf/pepper1.0_generated_urdf/pepperTransmission.xacro (robot description, xacro)
@@ -85,5 +85,5 @@
 			</actuator>
 		</transmission>
-		<transmission name="${side}Hand_Transmission">
+<!-- 		<transmission name="${side}Hand_Transmission">
 			<type>transmission_interface/SimpleTransmission</type>
 			<joint name="${side}Hand">
@@ -94,5 +94,5 @@
 				<mechanicalReduction>${speed_red_type3B}</mechanicalReduction>
 			</actuator>
-		</transmission>
+		</transmission> -->
 		</xacro:macro>
 	<xacro:arm_joints_transmissions side="L"/>

Commit message: Full config for the plugin
and cleanup warnings about transmissions

File: pepper_description/urdf/pepper1.0_generated_urdf/pepperGazebo.xacro (robot description, xacro)
@@ -691,18 +691,37 @@
 </gazebo>
 <!-- Drive controller -->
-  <gazebo>
-      <plugin name="base_drive_controller" filename="libgazebo_ros_model_velocity.so">
-          <robotNamespace>/pepper</robotNamespace>
-          <commandTopic>cmd_vel</commandTopic>
-          <updateRate>50.0</updateRate>
-          <!-- To simulate closer to the real robot we modified the
-          theoretical limits -->
-          <linearVelocityLimit>${0.55 * 1.0}</linearVelocityLimit>
-          <angularVelocityLimit>${2.0 * 1.0}</angularVelocityLimit>
-          <linearAccelerationLimit>${0.55 * 0.8}</linearAccelerationLimit>
-          <angularAccelerationLimit>${3.0 * 0.8}</angularAccelerationLimit>
-          <linearJerkLimit>${5.0 * 0.9}</linearJerkLimit>
-          <angularJerkLimit>${50.0 * 0.9}</angularJerkLimit>
-      </plugin>
-  </gazebo>
+<gazebo>
+  <plugin name="base_drive_controller" filename="libgazebo_ros_model_velocity.so">
+      <robotNamespace>/pepper</robotNamespace>
+      <commandTopic>cmd_vel</commandTopic>
+      <outputVelocityTopic>output_vel</outputVelocityTopic>
+      <updateRate>50.0</updateRate>
+      <commandTimeout>0.5</commandTimeout>
+      <!-- Publish odometry as needed -->
+      <odometryTopic>odom</odometryTopic>
+      <odometryFrame>odom</odometryFrame>
+      <odometryRate>20.0</odometryRate>
+      <publishOdometryTf>true</publishOdometryTf>
+      <robotBaseFrame>base_footprint</robotBaseFrame>
+      <!-- As measured in real robot odom_alpha3 and odom_alpha1 -->
+      <gaussianNoiseXY>0.02</gaussianNoiseXY>
+      <gaussianNoiseYaw>0.02645</gaussianNoiseYaw>
+      <!-- To simulate closer to the real robot we modified the
+      theoretical limits -->
+      <linearVelocityLimit>${0.55 * 1.0}</linearVelocityLimit>
+      <angularVelocityLimit>${2.0 * 1.0}</angularVelocityLimit>
+      <linearAccelerationLimit>${0.55 * 0.8}</linearAccelerationLimit>
+      <angularAccelerationLimit>${3.0 * 0.8}</angularAccelerationLimit>
+      <linearJerkLimit>${5.0 * 0.9}</linearJerkLimit>
+      <angularJerkLimit>${50.0 * 0.9}</angularJerkLimit>
+  </plugin>
+</gazebo>
+<gazebo>
+  <plugin name="ground_truth" filename="libgazebo_ros_p3d.so">
+    <frameName>world</frameName>
+    <bodyName>base_footprint</bodyName>
+    <topicName>/pepper/odom_groundtruth</topicName>
+    <updateRate>20.0</updateRate>
+  </plugin>
+</gazebo>
 </robot>

File: pepper_description/urdf/pepper1.0_generated_urdf/pepperTransmission.xacro (robot description, xacro)
@@ -13,9 +13,7 @@
 		<type>transmission_interface/SimpleTransmission</type>
 		<joint name="HeadYaw">
-        	<hardwareInterface>PositionJointInterface</hardwareInterface>
+        	<hardwareInterface>hardware_interface/PositionJointInterface</hardwareInterface>
 		</joint>
         <actuator name="HeadYaw_Motor">
-			<!-- Dummy Values -->
-			<hardwareInterface>PositionJointInterface</hardwareInterface>
 			<mechanicalReduction>${speed_red_type1A}</mechanicalReduction>
 		</actuator>
@@ -24,9 +22,7 @@
 		<type>transmission_interface/SimpleTransmission</type>
 		<joint name="HeadPitch">
-            <hardwareInterface>PositionJointInterface</hardwareInterface>
+            <hardwareInterface>hardware_interface/PositionJointInterface</hardwareInterface>
         </joint>
 		<actuator name="HeadPitch_Motor">
-			<!-- Dummy Values -->
-			<hardwareInterface>PositionJointInterface</hardwareInterface>
 			<mechanicalReduction>${speed_red_type2A}</mechanicalReduction>
 		</actuator>
@@ -38,8 +34,7 @@
 			<type>transmission_interface/SimpleTransmission</type>
 			<joint name="${side}ShoulderPitch">
-              <hardwareInterface>PositionJointInterface</hardwareInterface>
+              <hardwareInterface>hardware_interface/PositionJointInterface</hardwareInterface>
             </joint>
 			<actuator name="${side}ShoulderPitch_Motor">
-				<hardwareInterface>PositionJointInterface</hardwareInterface>
 				<mechanicalReduction>${speed_red_type1A}</mechanicalReduction>
 			</actuator>
@@ -48,8 +43,7 @@
 			<type>transmission_interface/SimpleTransmission</type>
 			<joint name="${side}ShoulderRoll">
-     			<hardwareInterface>PositionJointInterface</hardwareInterface>
+     			<hardwareInterface>hardware_interface/PositionJointInterface</hardwareInterface>
             </joint>
 			<actuator name="${side}ShoulderRoll_Motor">
-				<hardwareInterface>PositionJointInterface</hardwareInterface>
 				<mechanicalReduction>${speed_red_type2A}</mechanicalReduction>
 			</actuator>
@@ -58,8 +52,7 @@
 			<type>transmission_interface/SimpleTransmission</type>
 			<joint name="${side}ElbowYaw">
-              <hardwareInterface>PositionJointInterface</hardwareInterface>
+              <hardwareInterface>hardware_interface/PositionJointInterface</hardwareInterface>
             </joint>
 			<actuator name="${side}ElbowYaw_Motor">
-				<hardwareInterface>PositionJointInterface</hardwareInterface>
 				<mechanicalReduction>${speed_red_type1A}</mechanicalReduction>
 			</actuator>
@@ -68,8 +61,7 @@
 			<type>transmission_interface/SimpleTransmission</type>
 			<joint name="${side}ElbowRoll">
-    			<hardwareInterface>PositionJointInterface</hardwareInterface>
+    			<hardwareInterface>hardware_interface/PositionJointInterface</hardwareInterface>
             </joint>
 			<actuator name="${side}ElbowRoll_Motor">
-				<hardwareInterface>PositionJointInterface</hardwareInterface>
 				<mechanicalReduction>${speed_red_type2A}</mechanicalReduction>
 			</actuator>
@@ -78,18 +70,17 @@
 			<type>transmission_interface/SimpleTransmission</type>
 			<joint name="${side}WristYaw">
-              <hardwareInterface>PositionJointInterface</hardwareInterface>
+              <hardwareInterface>hardware_interface/PositionJointInterface</hardwareInterface>
             </joint>
 			<actuator name="${side}WristYaw_Motor">
-				<hardwareInterface>PositionJointInterface</hardwareInterface>
 				<mechanicalReduction>${speed_red_type2A}</mechanicalReduction>
 			</actuator>
 		</transmission>
+        <!-- Disabling hands as they cant do much in simulation anyways -->
 <!-- 		<transmission name="${side}Hand_Transmission">
 			<type>transmission_interface/SimpleTransmission</type>
 			<joint name="${side}Hand">
-  			  <hardwareInterface>PositionJointInterface</hardwareInterface>
+  			  <hardwareInterface>hardware_interface/PositionJointInterface</hardwareInterface>
             </joint>
 			<actuator name="${side}Hand_Motor">
-				<hardwareInterface>PositionJointInterface</hardwareInterface>
 				<mechanicalReduction>${speed_red_type3B}</mechanicalReduction>
 			</actuator>
@@ -102,9 +93,7 @@
 		<type>transmission_interface/SimpleTransmission</type>
 		<joint name="HipRoll">
-		  <hardwareInterface>PositionJointInterface</hardwareInterface>
+		  <hardwareInterface>hardware_interface/PositionJointInterface</hardwareInterface>
            </joint>
 		<actuator name="HipRoll_Motor">
-			<!-- Dummy Values -->
-			<hardwareInterface>PositionJointInterface</hardwareInterface>
 			<mechanicalReduction>${speed_red_type4A}</mechanicalReduction>
 		</actuator>
@@ -113,9 +102,7 @@
 		<type>transmission_interface/SimpleTransmission</type>
 		<joint name="HipPitch">
-		  <hardwareInterface>PositionJointInterface</hardwareInterface>
+		  <hardwareInterface>hardware_interface/PositionJointInterface</hardwareInterface>
            </joint>
 		<actuator name="HipPitch_Motor">
-			<!-- Dummy Values -->
-			<hardwareInterface>PositionJointInterface</hardwareInterface>
 			<mechanicalReduction>${speed_red_type5A}</mechanicalReduction>
 		</actuator>
@@ -124,14 +111,13 @@
 		<type>transmission_interface/SimpleTransmission</type>
 		<joint name="KneePitch">
-       		<hardwareInterface>PositionJointInterface</hardwareInterface>
+       		<hardwareInterface>hardware_interface/PositionJointInterface</hardwareInterface>
            </joint>
                 <actuator name="KneePitch_Motor">
-                        <!-- Dummy Values -->
-                        <hardwareInterface>PositionJointInterface</hardwareInterface>
                         <mechanicalReduction>${speed_red_type5A}</mechanicalReduction>
                 </actuator>
         </transmission>
         <!-- XACRO -->
-        <xacro:macro name="wheel_joints_transmissions" params="side">
+        <!-- Disabling wheels, given they are not used in simulation anymore -->
+<!--         <xacro:macro name="wheel_joints_transmissions" params="side">
                 <transmission name="Wheel${side}_Transmission">
                         <type>transmission_interface/SimpleTransmission</type>
@@ -140,6 +126,4 @@
                         </joint>
                         <actuator name="Wheel${side}_Motor">
-                                <!-- Dummy Values -->
-                                <hardwareInterface>EffortJointInterface</hardwareInterface>
                                 <mechanicalReduction>${speed_red_type5B}</mechanicalReduction>
                         </actuator>
@@ -148,4 +132,4 @@
         <xacro:wheel_joints_transmissions side="FL"/>
         <xacro:wheel_joints_transmissions side="B"/>
-        <xacro:wheel_joints_transmissions side="FR"/>
+        <xacro:wheel_joints_transmissions side="FR"/> -->
 </robot>

Commit message: Make the lasers works

File: pepper_description/urdf/pepper1.0_generated_urdf/pepperGazebo.xacro (robot description, xacro)
@@ -503,5 +503,5 @@
       <sensor type="depth" name="CameraDepth_frame_sensor">
         <always_on>true</always_on>
-        <update_rate>20.0</update_rate>
+        <update_rate>30.0</update_rate>
         <camera>
           <horizontal_fov>${58.0*3.14159265359/180.0}</horizontal_fov>
@@ -516,7 +516,9 @@
           </clip>
         </camera>
+        <!-- TODO: Fork our own https://github.com/ros-simulation/gazebo_ros_pkgs/blob/kinetic-devel/gazebo_plugins/src/gazebo_ros_openni_kinect.cpp#L396
+        to have the depth image be the same format -->
         <plugin name="CameraDepth_frame_controller" filename="libgazebo_ros_openni_kinect.so">
           <alwaysOn>true</alwaysOn>
-          <updateRate>20.0</updateRate>
+          <updateRate>30.0</updateRate>
           <cameraName>pepper/camera</cameraName>
           <imageTopicName>ir/image_raw</imageTopicName>
@@ -725,3 +727,131 @@
   </plugin>
 </gazebo>
+  <!-- Front -->
+  <gazebo reference="SurroundingFrontLaser_frame">
+    <sensor type="gpu_ray" name="front_laser_sensor">
+      <pose>0 0 0 0 0 0</pose>
+      <visualize>true</visualize>
+      <update_rate>6.25</update_rate>
+      <ray>
+        <scan>
+          <horizontal>
+            <samples>15</samples>
+            <resolution>1</resolution>
+            <min_angle>-0.5235987755982988</min_angle>
+            <max_angle>0.5235987755982988</max_angle>
+          </horizontal>
+        </scan>
+        <range>
+          <min>0.3</min>
+          <max>7.0</max>
+          <resolution>0.005</resolution>
+        </range>
+        <noise>
+          <type>gaussian</type>
+          <mean>0.01</mean>
+          <stddev>0.01</stddev>
+        </noise>
+      </ray>
+      <plugin name="gazebo_ros_front_laser_controller" filename="libgazebo_ros_gpu_laser.so">
+        <topicName>/pepper/scan_front</topicName>
+        <frameName>SurroundingFrontLaser_frame</frameName>
+      </plugin>
+    </sensor>
+  </gazebo>
+    <!-- Left -->
+  <gazebo reference="SurroundingLeftLaser_frame">
+    <sensor type="gpu_ray" name="left_laser_sensor">
+      <pose>0 0 0 0 0 0</pose>
+      <visualize>true</visualize>
+      <update_rate>6.25</update_rate>
+      <ray>
+        <scan>
+          <horizontal>
+            <samples>15</samples>
+            <resolution>1</resolution>
+            <min_angle>-0.5235987755982988</min_angle>
+            <max_angle>0.5235987755982988</max_angle>
+          </horizontal>
+        </scan>
+        <range>
+          <min>0.3</min>
+          <max>7.0</max>
+          <resolution>0.005</resolution>
+        </range>
+        <noise>
+          <type>gaussian</type>
+          <mean>0.01</mean>
+          <stddev>0.01</stddev>
+        </noise>
+      </ray>
+      <plugin name="gazebo_ros_left_laser_controller" filename="libgazebo_ros_gpu_laser.so">
+        <topicName>/pepper/scan_left</topicName>
+        <frameName>SurroundingLeftLaser_frame</frameName>
+      </plugin>
+    </sensor>
+  </gazebo>
+    <!-- Right -->
+  <gazebo reference="SurroundingRightLaser_frame">
+    <sensor type="gpu_ray" name="right_laser_sensor">
+      <pose>0 0 0 0 0 0</pose>
+      <visualize>true</visualize>
+      <update_rate>6.25</update_rate>
+      <ray>
+        <scan>
+          <horizontal>
+            <samples>15</samples>
+            <resolution>1</resolution>
+            <min_angle>-0.5235987755982988</min_angle>
+            <max_angle>0.5235987755982988</max_angle>
+          </horizontal>
+        </scan>
+        <range>
+          <min>0.3</min>
+          <max>7.0</max>
+          <resolution>0.005</resolution>
+        </range>
+        <noise>
+          <type>gaussian</type>
+          <mean>0.01</mean>
+          <stddev>0.01</stddev>
+        </noise>
+      </ray>
+      <plugin name="gazebo_ros_right_laser_controller" filename="libgazebo_ros_gpu_laser.so">
+        <topicName>/pepper/scan_right</topicName>
+        <frameName>SurroundingRightLaser_frame</frameName>
+      </plugin>
+    </sensor>
+  </gazebo>
+  <!-- Front -->
+  <gazebo reference="SurroundingFrontLaser_fake_hokuyo_frame">
+    <sensor type="gpu_ray" name="fake_hokuyo_laser_sensor">
+      <pose>0 0 0 0 0 0</pose>
+      <visualize>false</visualize>
+      <update_rate>6.25</update_rate>
+      <ray>
+        <scan>
+          <horizontal>
+            <samples>720</samples>
+            <resolution>1</resolution>
+            <min_angle>-1.570796</min_angle>
+            <max_angle>1.570796</max_angle>
+          </horizontal>
+        </scan>
+        <range>
+          <min>0.1</min>
+          <max>30.0</max>
+          <resolution>0.01</resolution>
+        </range>
+        <noise>
+          <type>gaussian</type>
+          <mean>0.0</mean>
+          <stddev>0.01</stddev>
+        </noise>
+      </ray>
+      <plugin name="gazebo_ros_fake_hokuyo_laser_controller" filename="libgazebo_ros_gpu_laser.so">
+        <topicName>/pepper/hokuyo_scan</topicName>
+        <frameName>SurroundingFrontLaser_fake_hokuyo_frame</frameName>
+      </plugin>
+    </sensor>
+  </gazebo>
 </robot>

File: pepper_description/urdf/pepper1.0_generated_urdf/pepper_sensors.xacro (robot description, xacro)
@@ -225,3 +225,10 @@
 		<axis xyz="0 0 0"/>
 	</joint>
+	<link name="SurroundingFrontLaser_fake_hokuyo_frame"/>
+	<joint name="LaserSensor/Front_fake_hokuyo_projected_sensor_fixedjoint" type="fixed">
+		<parent link="Tibia"/>
+		<child link="SurroundingFrontLaser_fake_hokuyo_frame"/>
+		<origin rpy="0 0 0" xyz="0.0562 0 -0.334"/>
+		<axis xyz="0 0 0"/>
+	</joint>
 </robot>
