Commit message: Fixing the robot model again... the lasers were in the wrong place...

File: pepper_description/urdf/pepper1.0_generated_urdf/pepper_sensors.xacro (robot description, xacro)
@@ -55,5 +55,5 @@
 		<parent link="Tibia"/>
 		<child link="SurroundingLeftLaser_frame"/>
-		<origin rpy="0 0 1.75728" xyz="-0.018 0.0899 -0.334"/>
+		<origin rpy="0 0 1.5707963267948966" xyz="-0.08600 0.10100 -0.30000"/>
 		<axis xyz="0 0 0"/>
 	</joint>
@@ -125,5 +125,5 @@
 		<parent link="Tibia"/>
 		<child link="SurroundingRightLaser_frame"/>
-		<origin rpy="0 0 -1.75728" xyz="-0.018 -0.0899 -0.334"/>
+		<origin rpy="0 0 -1.5707963267948966" xyz="-0.08600 -0.10100 -0.30000"/>
 		<axis xyz="0 0 0"/>
 	</joint>
@@ -208,5 +208,5 @@
 		<parent link="Tibia"/>
 		<child link="SurroundingFrontLaser_frame"/>
-		<origin rpy="0 0 0" xyz="0.0562 0 -0.334"/>
+		<origin rpy="0 0 0" xyz="0.12960 -0.02700 -0.30010"/>
 		<axis xyz="0 0 0"/>
 	</joint>
