Commit message: No more error at launch

File: pepper_description/urdf/pepper1.0_generated_urdf/pepperTransmission.xacro (robot description, xacro)
@@ -119,17 +119,17 @@
         <!-- XACRO -->
         <!-- Disabling wheels, given they are not used in simulation anymore -->
-<!--         <xacro:macro name="wheel_joints_transmissions" params="side">
-                <transmission name="Wheel${side}_Transmission">
-                        <type>transmission_interface/SimpleTransmission</type>
-                        <joint name="Wheel${side}">
-                                <hardwareInterface>EffortJointInterface</hardwareInterface>
-                        </joint>
-                        <actuator name="Wheel${side}_Motor">
-                                <mechanicalReduction>${speed_red_type5B}</mechanicalReduction>
-                        </actuator>
-                </transmission>
+        <xacro:macro name="wheel_joints_transmissions" params="side">
+            <transmission name="Wheel${side}_Transmission">
+				<type>transmission_interface/SimpleTransmission</type>
+				<joint name="Wheel${side}">
+						<hardwareInterface>EffortJointInterface</hardwareInterface>
+				</joint>
+				<actuator name="Wheel${side}_Motor">
+						<mechanicalReduction>${speed_red_type5B}</mechanicalReduction>
+				</actuator>
+            </transmission>
         </xacro:macro>
         <xacro:wheel_joints_transmissions side="FL"/>
         <xacro:wheel_joints_transmissions side="B"/>
-        <xacro:wheel_joints_transmissions side="FR"/> -->
+        <xacro:wheel_joints_transmissions side="FR"/>
 </robot>

File: pepper_description/urdf/pepper1.0_generated_urdf/pepperTransmission_no_arms.xacro (robot description, xacro)
@@ -119,17 +119,17 @@
         <!-- XACRO -->
         <!-- Disabling wheels, given they are not used in simulation anymore -->
-<!--         <xacro:macro name="wheel_joints_transmissions" params="side">
-                <transmission name="Wheel${side}_Transmission">
-                        <type>transmission_interface/SimpleTransmission</type>
-                        <joint name="Wheel${side}">
-                                <hardwareInterface>EffortJointInterface</hardwareInterface>
-                        </joint>
-                        <actuator name="Wheel${side}_Motor">
-                                <mechanicalReduction>${speed_red_type5B}</mechanicalReduction>
-                        </actuator>
-                </transmission>
+        <xacro:macro name="wheel_joints_transmissions" params="side">
+			<transmission name="Wheel${side}_Transmission">
+			<type>transmission_interface/SimpleTransmission</type>
+			<joint name="Wheel${side}">
+				<hardwareInterface>EffortJointInterface</hardwareInterface>
+			</joint>
+			<actuator name="Wheel${side}_Motor">
+				<mechanicalReduction>${speed_red_type5B}</mechanicalReduction>
+			</actuator>
+			</transmission>
         </xacro:macro>
         <xacro:wheel_joints_transmissions side="FL"/>
         <xacro:wheel_joints_transmissions side="B"/>
-        <xacro:wheel_joints_transmissions side="FR"/> -->
+        <xacro:wheel_joints_transmissions side="FR"/>
 </robot>

File: pepper_description/urdf/pepper1.0_generated_urdf/pepper_visual_collisions.xacro (robot description, xacro)
@@ -543,13 +543,13 @@
 		<visual>
 			<geometry>
-				<mesh filename="package://pepper_description/meshes/Torso.dae" scale="0.1 0.1 0.1"/>
-			</geometry>
-			<origin rpy="0 0 0" xyz="0 0 0"/>
-		</visual>
-		<collision>
-			<geometry>
 				<mesh filename="package://pepper_description/meshes/Torso_0.10.stl" scale="0.1 0.1 0.1"/>
 			</geometry>
 			<origin rpy="0 0 0" xyz="0 0 0"/>
+		</visual>
+		<collision>
+			<geometry>
+				<mesh filename="package://pepper_description/meshes/Torso_0.10.stl" scale="0.1 0.1 0.1"/>
+			</geometry>
+			<origin rpy="0 0 0" xyz="0 0 0"/>
 		</collision>
 	</xacro:macro>
